File: eagle/Node base/schematic.sch (EAGLE design)
At the start: 12 parts, among them IC1 MEGA8-AI, Q1 8MHz

Commit message: add tx/rx leds, finish adding connector, start board layout
Parts:
- removed HDR: 2526-5, con-3m:2526-5
- removed PWR: 236-412, con-wago-508:236-412
- added C4: 22pF, resistor:C-EUC0603
- added JP1: (no value), SparkFun-Passives:JUMPER-2PTH
- added JP2: (no value), pinhead:PINHD-1X22/90
- added R3, R5, R6, R7, R8, R9: 470, resistor:R-EU_R0603
- added RXLED, TXLED: (no value), led:LED
- added S1: (no value), switch-omron:10-XX
- C1, C2, C3, IC1, MCP2515, MCP2551, Q1, R1, R2: OC_NEWARK (none) -> unknown
Connections:
- removed net N$11: IC1.PC6(/RESET), ISP.1, R1.1
- removed net N$8: MCP2515D.RXCAN, MCP2551G$1.RXD
- new net N$13: R3.1, S1.S1
- new net N$14: IC1.PB0(ICP), MCP2515D.INT
- new net N$15: ISP.2, R5.2
- new net N$16: ISP.3, R6.2
- new net N$17: ISP.4, R7.2
- new net N$18: R8.1, TXLED.A
- new net N$19: R9.1, RXLED.A
- new net RESET: IC1.PC6(/RESET), ISP.1, JP2.17, R1.1, S1.P1
- new net RXLED: MCP2515D.RXCAN, MCP2551G$1.RXD, RXLED.C
- net GND: now also C4.2, JP1.2, JP2.22, R3.2
- net N$1: now also JP2.20, R7.1; no longer ISP.4
- net N$2: now also JP2.18, R6.1; no longer ISP.3
- net N$3: now also JP2.19, R5.1; no longer ISP.2
- net N$7: now also TXLED.C
- net PC0: now also JP2.1; no longer HDR-26.KL
- net PC1: now also JP2.2; no longer HDR-25.KL
- net PC2: now also JP2.3; no longer HDR-24.KL
- net PC3: now also JP2.4; no longer HDR-23.KL
- net PC4: now also JP2.5; no longer HDR-22.KL
- net PC5: now also JP2.6; no longer HDR-21.KL
- net PC6: now also JP2.7; no longer HDR-20.KL
- net PC7: now also JP2.8; no longer HDR-19.KL
- net PD0: now also JP2.9; no longer HDR-18.KL
- net PD1: now also JP2.10; no longer HDR-17.KL
- net PD2: now also JP2.11; no longer HDR-16.KL
- net PD3: now also JP2.12; no longer HDR-15.KL
- net PD4: now also JP2.13; no longer HDR-14.KL
- net PD5: now also JP2.14; no longer HDR-13.KL
- net PD6: now also JP2.15; no longer HDR-12.KL
- net PD7: now also JP2.16; no longer HDR-11.KL
- net VCC: now also C4.1, JP1.1, JP2.21, R8.2, R9.2
Other:
- moved on the sheet: ISP
