File: eagle/Node CPU/rev1.sch (EAGLE design)
At the start: 18 parts, among them IC1 MEGA8-AI, Q1 8MHz

Commit message: finished rev 1 of node CPU board
Parts:
- removed HDR: 2526-5, con-3m:2526-5
- removed MCP2515: (no value), can:MCP2515P
- removed MCP2551: MCP2551DIL8, can:MCP2551DIL8
- removed PWR: 236-412, con-wago-508:236-412
- removed R7: 470, resistor:R-EU_R0603
- added $$R7, R4, R8: 470, resistor:R-EU_R0603
- added JP1, JP11, JP12, JP13, JP14, JP15, JP16, JP17, JP18, JP19, JP2, JP20, JP21, JP22, JP23, JP3, JP4, JP5, JP6, JP7, JP8, JP9: (no value), pinhead:PINHD-1X1
- added JP10: (no value), SparkFun-Passives:JUMPER-2PTH
- added LED1, LED2: (no value), led:LEDCHIP-LED0603
- added MCP1: (no value), can:MCP2515P
- added MCP2: MCP2551DIL8, can:MCP2551DIL8
- added X1: (no value), con-wago-500:W237-102
- C1: value 22pF -> 0.1uF; OC_NEWARK (none) -> unknown
- C2, C4, IC1, Q1, R3: OC_NEWARK (none) -> unknown
- C3: value 0.1uF -> 22pF; OC_NEWARK (none) -> unknown
- R1, R2: value 10K -> 470; OC_NEWARK (none) -> unknown
- R5, R6: value 470 -> 10K; OC_NEWARK (none) -> unknown
Connections:
- removed net N$11: HDR-10.KL, IC1.PC6(/RESET), R1.1, S1.P1
- removed net N$6: ISP.1
- removed net N$8: MCP2515D.RXCAN, MCP2551G$1.RXD
- removed net PC0: HDR-26.KL, IC1.PC0(ADC0)
- removed net PC1: HDR-25.KL, IC1.PC1(ADC1)
- removed net PC2: HDR-24.KL, IC1.PC2(ADC2)
- removed net PC3: HDR-23.KL, IC1.PC3(ADC3)
- removed net PC4: HDR-22.KL, IC1.PC4(ADC4/SDA)
- removed net PC5: HDR-21.KL, IC1.PC5(ADC5/SCL)
- removed net PC6: HDR-20.KL, IC1.ADC6
- removed net PC7: HDR-19.KL, IC1.ADC7
- removed net PD0: HDR-18.KL, IC1.PD0(RXD)
- removed net PD1: HDR-17.KL, IC1.PD1(TXD)
- removed net PD2: HDR-16.KL, IC1.PD2(INT0)
- removed net PD3: HDR-15.KL, IC1.PD3(INT1)
- removed net PD4: HDR-14.KL, IC1.PD4(XCK/T0)
- removed net PD5: HDR-13.KL, IC1.PD5(T1)
- removed net PD6: HDR-12.KL, IC1.PD6(AIN0)
- removed net PD7: HDR-11.KL, IC1.PD7(AIN1)
- new net N$18: LED2.A, R8.1
- new net N$19: $$R7.1, LED1.A
- new net N$20: IC1.PC0(ADC0), JP3.1
- new net N$21: IC1.PC1(ADC1), JP2.1
- new net N$22: IC1.PC2(ADC2), JP1.1
- new net N$23: IC1.PC3(ADC3), JP9.1
- new net N$24: IC1.PC4(ADC4/SDA), JP13.1
- new net N$25: IC1.PC5(ADC5/SCL), JP15.1
- new net N$26: IC1.ADC6, JP5.1
- new net N$27: IC1.ADC7, JP4.1
- new net N$28: IC1.PD0(RXD), JP18.1
- new net N$29: IC1.PD1(TXD), JP19.1
- new net N$30: IC1.PD2(INT0), JP20.1
- new net N$31: IC1.PD3(INT1), JP21.1
- new net N$32: IC1.PD4(XCK/T0), JP22.1
- new net N$33: IC1.PD5(T1), JP23.1
- new net N$34: IC1.PD6(AIN0), JP14.1
- new net N$35: IC1.PD7(AIN1), JP12.1
- new net N$36: MCP2G$1.CANL, X1-2.KL
- new net N$37: MCP2G$1.CANH, X1-1.KL
- new net RESET: IC1.PC6(/RESET), ISP.1, JP8.1, R5.1, S1.P, S1.P1
- new net RXLED: LED1.C, MCP1D.RXCAN, MCP2G$1.RXD
- net GND: now also C1.2, C2.2, C3.1, JP10.2, JP17.1, MCP2G$1.RS, R1.2; no longer C1.1, C2.1, C3.2, MCP2551G$1.RS, R3.2
- net N$1: now also JP6.1, MCP1D.SCK, R2.1; no longer HDR-7.KL, MCP2515D.SCK, R7.1
- net N$10: now also C3.2; no longer C2.2
- net N$12: now also MCP1D.RESET, R6.1; no longer MCP2515D.RESET, R2.1
- net N$13: now also R1.1, S1.S; no longer R3.1
- net N$14: now also MCP1D.INT; no longer MCP2515D.INT
- net N$15: now also R4.2; no longer R5.2
- net N$16: now also R3.2; no longer R6.2
- net N$17: now also R2.2; no longer R7.2
- net N$2: now also JP11.1, MCP1D.SO, R3.1; no longer HDR-9.KL, MCP2515D.SO, R6.1
- net N$3: now also JP7.1, MCP1D.SI, R4.1; no longer HDR-8.KL, MCP2515D.SI, R5.1
- net N$4: now also MCP1D.CS; no longer MCP2515D.CS
- net N$5: now also MCP1D.OSC1; no longer MCP2515D.OSC1
- net N$7: now also LED2.C, MCP1D.TXCAN, MCP2G$1.TXD; no longer MCP2515D.TXCAN, MCP2551G$1.TXD
- net N$9: now also C4.2; no longer C1.2
- net VCC: now also $$R7.2, C1.1, C2.1, JP10.1, JP16.1, R5.2, R6.2, R8.2; no longer C3.1, C4.2, R1.2, R2.2
Other:
- moved on the sheet: C1, C2, C3, C4, ISP, R1, R2, R3, R5, R6
