File: eagle/Node CPU/rev2.brd (EAGLE design)
At the start: 50 x 50 mm, 44 parts, among them IC1 MEGA8-AI

Commit message: updated to revision 3 of the board
Parts:
- moved R5 25.4 mm to (9.85, 24.5)
- moved MISO 7.62 mm to (48.0, 40.1)
- moved MOSI 7.62 mm to (48.0, 32.5)
- moved R2 5.49 mm to (27.9, 41.4)
- moved R4 5.44 mm to (22.9, 41.4)
- moved ISP 5.08 mm to (25.3, 38.1)
- moved R3 2.07 mm to (25.4, 41.4)
- moved R1 2.07 mm to (20.2, 41.4), turned to 270 degrees
- moved PWR 1.02 mm to (9.91, 21.3)
Connections:
- removed net N$1: IC1.17, MCP1.13, R2.1, SCK.1
- removed net N$16: ISP.3, R3.2
- new net N$38: MCP1.15, MISO.1, R3.2
- new net N$39: IC1.17, ISP.4, R4.1
- net N$15: now also MCP1.13, SCK.1; no longer ISP.2
- net N$17: now also IC1.15, ISP.2, R2.1; no longer ISP.4, R2.2
- net N$2: now also ISP.3; no longer MCP1.15, MISO.1
- net N$3: now also R2.2; no longer IC1.15, R4.1
Routing:
- net N$38: track 0.00 -> 55.3 mm
- net N$1: track 47.1 -> 0.00 mm
- net N$2: track 54.0 -> 10.9 mm, vias 1 -> 0
- net N$15: track 2.96 -> 36.4 mm
- net VCC: track 137.5 -> 110.9 mm, vias 2 -> 1
- net GND: track 191.6 -> 173.8 mm
- net N$39: track 0.00 -> 8.99 mm
- net N$17: track 2.96 -> 11.9 mm
- net RESET: track 63.1 -> 71.8 mm
- net N$16: track 2.96 -> 0.00 mm
- net N$3: track 44.9 -> 42.9 mm
- net N$13: track 18.3 -> 19.9 mm
Other:
- board text added: "Node CPU Rev. 2"
- board text added: "Revision 2"
- board text removed: "Node CPU Rev. 1"
- board text removed: "Revision 1"
